Commit message: Add some nodes and urdf

File: urdf/rb5.urdf (robot description, URDF)
Before this commit: robot rb5_850e, 8 links, 7 joints
Links:
- added link rgbd_sensor; visual mesh filename=package://urdf/meshes/visual/???

Commit message: Moving Test

File: urdf/rb5.urdf (robot description, URDF)
Before this commit: robot rb5_850e, 9 links, 7 joints
Links:
- link link0: geometry collision mesh filename=package://rb5_ros_wrapper/urdf/meshes/collision/link0.stl; visual mesh filename=package://rb5_ros_wrapper/urdf/meshes/visual/link0.dae
- link link1: geometry collision mesh filename=package://rb5_ros_wrapper/urdf/meshes/collision/link1.stl; visual mesh filename=package://rb5_ros_wrapper/urdf/meshes/visual/link1.dae
- link link2: geometry collision mesh filename=package://rb5_ros_wrapper/urdf/meshes/collision/link2.stl; visual mesh filename=package://rb5_ros_wrapper/urdf/meshes/visual/link2.dae
- link link3: geometry collision mesh filename=package://rb5_ros_wrapper/urdf/meshes/collision/link3.stl; visual mesh filename=package://rb5_ros_wrapper/urdf/meshes/visual/link3.dae
- link link4: geometry collision mesh filename=package://rb5_ros_wrapper/urdf/meshes/collision/link4.stl; visual mesh filename=package://rb5_ros_wrapper/urdf/meshes/visual/link4.dae
- link link5: geometry collision mesh filename=package://rb5_ros_wrapper/urdf/meshes/collision/link5.stl; visual mesh filename=package://rb5_ros_wrapper/urdf/meshes/visual/link5.dae
- link link6: geometry collision mesh filename=package://rb5_ros_wrapper/urdf/meshes/collision/link6.stl; visual mesh filename=package://rb5_ros_wrapper/urdf/meshes/visual/link6.dae
- link rgbd_sensor: geometry visual box size=0.02 0.02 0.02
Joints:
- added joint rgbd_sensor_joint: type fixed, parent link6, child rgbd_sensor, origin xyz=0 0 0 rpy=0 0 0
